File: Hardware/v4/current_sense.sch (EAGLE design)
At the start: 39 parts, among them J1 SCREW-TERMINAL_2_0.100, J2 SCREW-TERMINAL_2_0.100, J3 SCREW-TERMINAL_2_0.100, J4 SCREW-TERMINAL_2_0.100, U1 MAX9923H, U2 LP3985

Commit message: v4: update attrs
Parts:
- C1: DESCRIPTION (none) -> CAP CER 10000PF 25V X7R 0603; MANUFACTURER (none) -> TDK; MPN (none) -> C1608X7R1E103K080AA
- C2: DESCRIPTION (none) -> CAP CER .10UF 25V X7R 10% 0603; MANUFACTURER (none) -> TDK; MPN (none) -> C1608X7R1E104K080AA
- C3, C4: DESCRIPTION (none) -> CAP CER 1UF 16V X7R 0603; MANUFACTURER (none) -> TDK; MPN (none) -> C1608X7R1C105K080AC
- R1: DESCRIPTION (none) -> RES 0.04 OHM 1% 1/4W 1206; MANUFACTURER (none) -> Yageo; MPN (none) -> RL1206FR-070R04L
- R2: DESCRIPTION (none) -> RES 0.12 OHM 1% 1/2W 1206; MANUFACTURER (none) -> Susumu; MPN (none) -> RL1632R-R120-F
- R3: DESCRIPTION (none) -> RES 0.2 OHM 1% 1/2W 1206; MANUFACTURER (none) -> Stackpole Electronics; MPN (none) -> CSR1206FKR200
- R4: DESCRIPTION (none) -> RES 0.4 OHM 1% 1/4W 1206; MANUFACTURER (none) -> Yageo; MPN (none) -> RL1206FR-070R4L
- R5: DESCRIPTION (none) -> RES SMD 1.2 OHM 1% 1/3W 0805; MANUFACTURER (none) -> Susumu; MPN (none) -> RL1220S-1R2-F
- R6: DESCRIPTION (none) -> RES SMD 12 OHM 0.1% 1/10W 0805; MANUFACTURER (none) -> TE Connectivity; MPN (none) -> CPF0805B12RE1
- R7: DESCRIPTION (none) -> RES SMD 120 OHM 0.05% 1/8W 0805; MANUFACTURER (none) -> Susumu; MPN (none) -> RG2012N-121-W-T1
- R8: DESCRIPTION (none) -> RES 1.0K OHM 1/10W .1% 0603 SMD; MANUFACTURER (none) -> Panasonic; MPN (none) -> ERA-3AEB102V
- R9: DESCRIPTION (none) -> RES 249K OHM 1/10W .1% 0603 SMD; MANUFACTURER (none) -> Panasonic; MPN (none) -> ERA-3AEB2493V
- S1: DESCRIPTION (none) -> SWITCH ROTARY 7POS 500MA 24V; MANUFACTURER (none) -> C&K Components; MPN (none) -> RM107772BCB
- U1: DESCRIPTION (none) -> IC AMP CURRENT SENSE 10-MSOP; MANUFACTURER (none) -> Maxim Integrated; MPN (none) -> MAX9922EUB+T
